Commit message: Check

File: rotors_sim/src/rotors_description/urdf/iris.xacro (robot description, xacro)
@@ -130,4 +130,5 @@
     <xacro:insert_block name="rotor_inertia" />
   </xacro:vertical_rotor>
+<!--
   <link name="${namespace}/box">
     <xacro:box_inertial x="-0.1" y="-0.1" z="-0.1" mass="0.2">
@@ -152,6 +153,12 @@
     <child link="${namespace}/box" />
   </joint>
+ -->
+<!--
 <xacro:velodyne name="${namespace}/lidar" parent="${namespace}/base_link">
   <origin xyz="0.0 0.0 0.2" rpy="0 0 0"/>
 </xacro:velodyne>
+ -->
+<xacro:kinect_module name="${namespace}/kinect" parent="${namespace}/base_link">
+  <origin xyz="0.2 0.0 0.05" rpy="0 0 0"/>
+</xacro:kinect_module>
 </robot>

File: rotors_sim/src/rotors_description/urdf/multirotor_base.xacro (robot description, xacro)
@@ -218,3 +218,87 @@
     <xacro:velodyne_sensor link_name="${name}" frame_name="${parent}" lidar_name="${name}" />
   </xacro:macro>
+  <xacro:macro name="kinect_module" params="name parent *origin">
+    <link name="${name}_link">
+      <inertial>
+        <mass value="0.01"/>
+        <origin xyz="0.0 0 0" rpy="0 0 0"/>
+        <inertia ixx="0.01" ixy="0.0" ixz="0.0" iyy="0.01" iyz="0.0" izz="0.01"/>
+      </inertial>
+      <collision name="collision">
+        <geometry>
+          <box size="0.073000 0.276000 0.072000" />
+        </geometry>
+      </collision>
+      <visual>
+        <geometry>
+          <mesh filename="package://rotors_description/meshes/kinect.dae" scale="1 1 1" />
+        </geometry>
+      </visual>
+      <sensor name="${name}_sensor" type="depth">
+        <update_rate>20</update_rate>
+        <camera>
+          <horizontal_fov>1.047198</horizontal_fov>
+          <image>
+            <width>640</width>
+            <height>480</height>
+            <format>R8G8B8</format>
+          </image>
+          <clip>
+            <near>0.01</near>
+            <far>5</far>
+          </clip>
+        </camera>
+      </sensor>
+    </link>
+    <link name="${name}_link_optical">
+    </link>
+    <joint name="camera_optical_joint" type="fixed">
+    <!-- these values have to be these values otherwise the gazebo camera
+        image won't be aligned properly with the frame it is supposedly
+        originating from -->
+      <origin xyz="0 0 0" rpy="${-pi/2} 0 ${-pi/2}"/>
+      <parent link="${name}_link"/>
+      <child link="${name}_link_optical"/>
+    </joint>
+    <joint name="${name}_joint" type="fixed">
+      <xacro:insert_block name="origin"/>
+      <parent link="${parent}"/>
+      <child link="${name}_link"/>
+    </joint>
+    <xacro:property name="link_name" value="${name}_link"/>
+    <xacro:property name="optical_link_name" value="${name}_link_optical"/>
+    <gazebo reference="${name}_link">
+      <sensor name="${name}_sensor" type="depth">
+      <!-- <sensor> -->
+        <!-- <plugin name="kinect_plugin" filename="libgazebo_ros_camera.so"> -->
+        <plugin name="camera_plugin" filename="libgazebo_ros_openni_kinect.so">
+          <baseline>0.2</baseline>
+          <alwaysOn>true</alwaysOn>
+          <!-- Keep this zero, update_rate in the parent <sensor> tag
+            will control the frame rate. -->
+          <updateRate>0.0</updateRate>
+          <cameraName>camera_ir</cameraName>
+          <imageTopicName>/iris/camera/color/image_raw</imageTopicName>
+          <cameraInfoTopicName>/iris/camera/color/camera_info</cameraInfoTopicName>
+          <depthImageTopicName>/iris/camera/depth/image_raw</depthImageTopicName>
+          <depthImageCameraInfoTopicName>/iris/camera/depth/camera_info</depthImageCameraInfoTopicName>
+          <pointCloudTopicName>/iris/camera/depth/points</pointCloudTopicName>
+          <frameName>kinect_link_optical</frameName>
+          <pointCloudCutoff>0.5</pointCloudCutoff>
+          <pointCloudCutoffMax>5.0</pointCloudCutoffMax>
+          <distortionK1>0</distortionK1>
+          <distortionK2>0</distortionK2>
+          <distortionK3>0</distortionK3>
+          <distortionT1>0</distortionT1>
+          <distortionT2>0</distortionT2>
+          <CxPrime>0</CxPrime>
+          <Cx>0</Cx>
+          <Cy>0</Cy>
+          <focalLength>0</focalLength>
+          <hackBaseline>0</hackBaseline>
+        </plugin>
+      </sensor>
+    </gazebo>
+    <!-- <xacro:kinect_sensor link_name="${name}" frame_name="{parent}"/>  -->
+  </xacro:macro>
 </robot>

File: rotors_sim/src/rotors_description/urdf/pelican.xacro (robot description, xacro)
@@ -23,9 +23,9 @@
   <xacro:property name="use_mesh_file" value="true" />
   <xacro:property name="mesh_file" value="package://rotors_description/meshes/pelican.dae" />
-  <xacro:property name="mass" value="1.0" /> <!-- [kg] -->
+  <xacro:property name="mass" value="1.63" /> <!-- [kg] -->
   <xacro:property name="body_width" value="0.1" /> <!-- [m] -->
   <xacro:property name="body_height" value="0.2" /> <!-- [m] -->
-  <xacro:property name="mass_rotor" value="0.01" /> <!-- [kg] -->
-  <xacro:property name="arm_length" value="0.21" /> <!-- [m] -->
+  <xacro:property name="mass_rotor" value="0.08" /> <!-- [kg] -->
+  <xacro:property name="arm_length" value="0.24" /> <!-- [m] -->
   <xacro:property name="rotor_offset_top" value="0.05" /> <!-- [m] -->
   <xacro:property name="radius_rotor" value="0.128" /> <!-- [m] -->
@@ -34,10 +34,10 @@
   <xacro:property name="time_constant_up" value="0.0125" /> <!-- [s] -->
   <xacro:property name="time_constant_down" value="0.025" /> <!-- [s] -->
-  <xacro:property name="max_rot_velocity" value="838" /> <!-- [rad/s] -->
+  <xacro:property name="max_rot_velocity" value="1838" /> <!-- [rad/s] -->
   <xacro:property name="rotor_drag_coefficient" value="8.06428e-05" />
   <xacro:property name="rolling_moment_coefficient" value="0.000001" />
   <!-- Property Blocks -->
   <xacro:property name="body_inertia">
-    <inertia ixx="0.01" ixy="0.0" ixz="0.0" iyy="0.01" iyz="0.0" izz="0.02" /> <!-- [kg m^2] [kg m^2] [kg m^2] [kg m^2] [kg m^2] [kg m^2] -->
+    <inertia ixx="0.016" ixy="0.0" ixz="0.0" iyy="0.016" iyz="0.0" izz="0.032" /> <!-- [kg m^2] [kg m^2] [kg m^2] [kg m^2] [kg m^2] [kg m^2] -->
   </xacro:property>
   <!-- inertia of a single rotor, assuming it is a cuboid. Height=3mm, width=15mm -->
